Commit message: week5

File: src/part2_robot_descriptions/urdf/robot2.xacro (robot description, xacro)
@@ -42,5 +42,11 @@
     </collision>
     <visual name="caster_front_visual">
-      <origin rpy=" 0 0 0" xyz="0.2 0 -0.05"/>
+      <origin rpy=" 0 0 0" xyz="0.4 0 -0.05"/>
+      <geometry>
+        <sphere radius="0.05"/>
+      </geometry>
+    </visual>
+    <visual name="caster_front_visual_2">
+      <origin rpy=" 0 0 0" xyz="-0.4 0 -0.05"/>
       <geometry>
         <sphere radius="0.05"/>

File: src/part2_robot_descriptions/urdf/robot3.xacro (robot description, xacro)
@@ -57,5 +57,5 @@
       <origin rpy="0 1.5707 1.5707" xyz="0 0 0"/>
       <geometry>
-        <cylinder length="0.04" radius="0.1707"/>
+        <cylinder length="0.04" radius="0.1"/>
       </geometry>
     </collision>

File: src/part2_robot_descriptions/urdf/robot4.xacro (robot description, xacro)
@@ -71,5 +71,5 @@
     <child link="link_right_wheel"/>
     <parent link="link_chassis"/>
-    <axis rpy="0 0 0" xyz="1 0 0"/>
+    <axis rpy="0 0 0" xyz="0 1 0"/>
     <limit effort="10000" velocity="1000"/>
     <joint_properties damping="1.0" friction="1.0"/>
@@ -98,5 +98,5 @@
     <child link="link_left_wheel"/>
     <parent link="link_chassis"/>
-    <axis rpy="0 0 0" xyz="1 0 0"/>
+    <axis rpy="0 0 0" xyz="0 1 0"/>
     <limit effort="10000" velocity="1000"/>
     <joint_properties damping="1.0" friction="1.0"/>
